File: pcb_rduhr_lderyck/pcb_rduhr_lderyck.kicad_sch (KiCad schematic)
At the start: 42 parts, among them J1 Conn_ARM_JTAG_SWD_10, J2 Résistance chauffante, Q1 NMOS, SW1 SW_DPDT_x2, U1 STM32F030F4Px, U2 AP7333, U3 MCP9700Ax-ETT, U4 MIC5271, Y1 Crystal_Small

Commit message: Carte uP quasi fini
Parts:
- removed C2: 1µF, Capacitor_SMD:C_0603_1608Metric_Pad1.08x0.95mm_HandSolder, symbol Device:C_Polarized
- added C14, C15: C, symbol Device:C
- added C2: 1uF, Capacitor_SMD:C_0603_1608Metric_Pad1.08x0.95mm_HandSolder, symbol Device:C
- added D4: D_Schottky, symbol Device:D_Schottky
- added J3: Conn_15_-15, symbol Connector:Conn_01x03_Pin
- added J4: Conn_1.8, symbol Connector:Conn_01x02_Pin
- added J5: Probe_15, symbol Connector:Conn_01x02_Pin
- added J6: Probe_-15, symbol Connector:Conn_01x02_Pin
- added J7: RX_TX, symbol Connector:Conn_01x02_Pin
- added J8: RF, symbol Connector:Conn_01x04_Pin
- added L1: L, symbol Device:L
- added Q2: NMOS, Package_TO_SOT_SMD:SOT-89-3, symbol Simulation_SPICE:NMOS
- added R11, R12, R13: R, symbol Device:R
- XC1: footprint (none) -> Package_TO_SOT_SMD:SOT-353_SC-70-5
Connections:
- net +15V: now also J3.1 (Pin_1), J5.1 (Pin_1); no longer C11.1, U2.1 (VI)
- net +3.3V: now also XC1. (VDD), C15.1, C2.1, R12.1, R13.1
- net +8V: now also J8.1 (Pin_1)
- net -15V: now also J3.2 (Pin_2), J6.1 (Pin_1); no longer C13.2, U4.1 (IN), U4.3 (EN)
- net -8V: now also J8.2 (Pin_2)
- net GND: now also XC1. (VDD), C15.2, C2.2, J3.3 (Pin_3), J4.2 (Pin_2), J8.4 (Pin_4), Q2.3 (S), R11.2
- new net: C14.2, R11.1, R13.2, XC1. (VDD)
- new net: Q2.2 (G), XC1. (VDD)
- new net: C14.1, D4.1 (K), R12.2
- new net: D4.2 (A), L1.2, Q2.1 (D)
- new net +1V8: J4.1 (Pin_1), L1.1
- new net Ap-15: C13.2, J6.2 (Pin_2), U4.1 (IN), U4.3 (EN)
- new net Ap15: C11.1, J5.2 (Pin_2), U2.1 (VI)
- new net CE: XC1. (VDD)
- new net DATA: J8.3 (Pin_3)
- new net RX: J7.1 (Pin_1)
- new net TX: J7.2 (Pin_2)
Other:
- moved on the sheet: C1, C10, C3, C4, C5, C6, C7, C8, D1, D2, D3, J1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

Commit message: Update PCB 1
Parts:
- removed R7: 4,7k, Resistor_SMD:R_0603_1608Metric_Pad0.98x0.95mm_HandSolder, symbol Device:R
- removed TP5, TP6: TestPoint, TestPoint:TestPoint_Pad_D1.5mm, symbol Connector:TestPoint
- removed Y1: Crystal_Small, Crystal:Crystal_SMD_HC49-SD_HandSoldering, symbol Device:Crystal_Small
- added C16, C17: 10uF, Capacitor_SMD:C_0603_1608Metric_Pad1.08x0.95mm_HandSolder, symbol Device:C
- added D5: LED, Diode_SMD:D_0603_1608Metric_Pad1.05x0.95mm_HandSolder, symbol Device:LED
- added Y1: Crystal, symbol Device:Crystal_GND24_Small
- C11, C12, C13, C14, C9: footprint (none) -> Capacitor_SMD:C_0603_1608Metric_Pad1.08x0.95mm_HandSolder
- C15: value C -> 10uF; footprint (none) -> Capacitor_SMD:C_0603_1608Metric_Pad1.08x0.95mm_HandSolder
- C4: value 1uF -> 4.7uF
- C6, C7: value 8pF -> 10pF
- R1: footprint Resistor_SMD:R_0603_1608Metric_Pad0.98x0.95mm_HandSolder -> (none)
- R10: value 560 ohm -> 5.6k
- R4, R5: value 1k -> 2.4k
- R6: value 4,7k -> 1k
- R8: value R -> 10k
- R9: value 100 ohm -> 1k
Connections:
- net CE is gone; now on net GND: XC1. (VDD)
- net +1V8: now also C16.1
- net +3.3V: now also C17.1
- net +8V: now also R4.1
- net -8V: now also R5.1
- net Ap-15: now also C13.1; no longer C13.2, U4.3 (EN)
- net GND: now also C13.2, D3.2 (A), C16.2, C17.2, D5.1 (K), Y1.2, Y1.4; no longer C13.1, D3.1 (K)
- net RX: now also U1.9 (PA3)
- net TEMP: now also U1.11 (PA5)
- net TX: now also U1.8 (PA2)
- net at R1.2, U1.2 (PF0): no longer C6.1
- net at R5.2: now also D3.1 (K); no longer D3.2 (A)
- net at C7.1, U1.3 (PF1): now also Y1.3; no longer R1.1
- net at Q1.2 (G), R8.1: now also U1.10 (PA4)
- net CE3.3: now reaches U1.12 (PA6)
- net CE3.3: now also XC1. (VDD)
- net CE-8: now reaches U1.13 (PA7)
- net CE-8: now also U4.3 (EN)
- net DATA renamed DEMOD
- net DEMOD: now also U1.7 (PA1)
- net LED1 renamed LED
- removed net LED2: R4.1, U1.7 (PA1)
- removed net LED3: R5.1, U1.8 (PA2)
- net SCL: no longer names the net of U1.17 (PA9)
- net SDA: no longer names the net of R6.2
- net SDA: now also D5.2 (A); no longer U1.18 (PA10)
- net SWO/TDO: no longer names the net of J1.6 (SWO/TDO)
- new net: C6.1, R1.1, Y1.1
Other:
- note removed: "HC49"
- note removed: "PULL-UP RESISTOR"
- moved on the sheet: C1, C10, C11, C12, C14, C15, C2, C3, C4, C5, C6, C7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

Commit message: Update pcb alim 2
Parts:
- removed TP7: TestPoint, TestPoint:TestPoint_Pad_D1.5mm, symbol Connector:TestPoint
- removed U2: AP7333, Package_TO_SOT_SMD:SOT-23, symbol Regulator_Linear:AP7384-28SA
- added C18: 10uF, Capacitor_SMD:C_0603_1608Metric_Pad1.08x0.95mm_HandSolder, symbol Device:C
- added JP1: SolderJumper, Jumper:SolderJumper-3_P1.3mm_Bridged12_Pad1.0x1.5mm, symbol Jumper:SolderJumper_3_Bridged12
- added R14: 10k, Resistor_SMD:R_0603_1608Metric_Pad0.98x0.95mm_HandSolder, symbol Device:R
- added R15: 1.1k, Resistor_SMD:R_0603_1608Metric_Pad0.98x0.95mm_HandSolder, symbol Device:R
- added R7: 200, Resistor_SMD:R_0603_1608Metric_Pad0.98x0.95mm_HandSolder, symbol Device:R
- added TP1, TP2: TestPoint, TestPoint:TestPoint_Pad_D1.5mm, symbol Connector:TestPoint
- added U5: LM1117, Package_TO_SOT_SMD:SOT-223-3_TabPin2, symbol Regulator_Linear:LM1117MP-ADJ
- C11, C9: value 1uF -> 10uF
- C14: value C -> 47pF
- D4: footprint (none) -> footprints:DO-214AC
- J2, J4, J5, J6, J7: footprint (none) -> Connector_PinSocket_2.54mm:PinSocket_1x02_P2.54mm_Vertical
- J3: footprint (none) -> Connector_PinSocket_2.54mm:PinSocket_1x03_P2.54mm_Vertical
- J8: footprint (none) -> Connector_PinSocket_2.54mm:PinSocket_1x04_P2.54mm_Vertical
- L1: value L -> 10uH; footprint (none) -> footprints:8.1_mm_x_7.3_mm_x_5.3_mm_Inductance
- Q1, Q2: footprint Package_TO_SOT_SMD:SOT-89-3 -> Package_TO_SOT_SMD:SOT-89-3_Handsoldering
- R1, R10, R8, R9: footprint (none) -> Resistor_SMD:R_0603_1608Metric_Pad0.98x0.95mm_HandSolder
- R11: value R -> 47k; footprint (none) -> Resistor_SMD:R_0603_1608Metric_Pad0.98x0.95mm_HandSolder
- R12: value R -> 0.1; footprint (none) -> Resistor_SMD:R_0603_1608Metric_Pad0.98x0.95mm_HandSolder
- R13: value R -> 120k; footprint (none) -> Resistor_SMD:R_0603_1608Metric_Pad0.98x0.95mm_HandSolder
- XC9103: renamed from XC1; footprint Package_TO_SOT_SMD:SOT-353_SC-70-5 -> footprints:SOT25
- Y1: footprint (none) -> Crystal:Crystal_SMD_3225-4Pin_3.2x2.5mm_HandSoldering
Connections:
- net +1V8: now also XC9103.2 (VDD), JP1.1 (A)
- net +3.3V: now also R14.1; no longer XC9103. (VDD)
- net +8V: now also R7.2, U5.2 (VO)
- net Ap15: now also U5.3 (VI)
- net CE-8: now also U1.12 (PA6); no longer U1.13 (PA7)
- net GND: now also XC9103.4 (GND), C18.2, JP1.3 (B), R15.1; no longer XC9103. (VDD)
- net RST: now also R14.2
- net TEMP: now also TP1.1
- net at C14.2, R11.1, R13.2: now also XC9103.1 (FB); no longer XC9103. (VDD)
- net at Q2.2 (G): now also XC9103.5 (EXT), TP2.1; no longer XC9103. (VDD)
- removed net CE3.3: U1.12 (PA6), XC9103. (VDD)
- new net: JP1.2 (C), XC9103.3 (CE)
- new net: C18.1, R15.2, R7.1, U5.1 (ADJ)
Other:
- moved on the sheet: C14, C15, C16, C17, D4, L1, Q2, R11, R12, R13, RST1, TP4
