File: uP_power_supply/pcb_rduhr_lderyck.kicad_pcb (KiCad board)
At the start: 2 copper layers, 62 parts, among them J1 Conn_ARM_JTAG_SWD_10, J2 Résistance chauffante, J3 Conn_15_-15, J4 Conn_1.8, J5 Probe_15, J6 Probe_-15, J7 RX_TX, J8 RF, Q1 NMOS, Q2 NMOS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

Commit message: PCB microp prêt pour impression !
Parts:
- moved JP1 212.3 mm to (76.2, 78.9), turned to 180 degrees
- moved TP2 211.8 mm to (74.3, 86.2), turned to 180 degrees
- moved C16 206.3 mm to (78.3, 82.0), turned to 0 degrees
- moved XC9103 206.2 mm to (77.5, 85.0), turned to 180 degrees
- moved R11 201.4 mm to (80.1, 84.7), turned to -90 degrees
- moved Q2 201.0 mm to (78.5, 91.5), turned to -90 degrees
- moved C14 197.7 mm to (82.0, 84.7), turned to 90 degrees
- moved R13 197.5 mm to (83.0, 81.8), turned to 180 degrees
- moved R12 194.0 mm to (83.9, 84.7), turned to -90 degrees
- moved C15 192.7 mm to (85.9, 80.9), turned to 90 degrees
- moved D4 190.8 mm to (84.3, 89.1), turned to 180 degrees
- moved C17 190.4 mm to (85.9, 84.6), turned to -90 degrees
- moved L1 183.8 mm to (86.5, 95.0), turned to -90 degrees
- moved C12 155.7 mm to (107.0, 93.3)
- moved C13 155.7 mm to (98.5, 93.3)
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Routing:
- net +3.3V: track 18.6 -> 103.6 mm, vias 0 -> 4
- net +15V: track 0.00 -> 46.4 mm, vias 0 -> 2
- net RST: track 9.34 -> 54.0 mm, vias 0 -> 2
- net Net-(Q1-G): track 2.53 -> 36.7 mm, vias 0 -> 4
- net +1V8: track 4.88 -> 38.6 mm
- net Ap15: track 2.38 -> 35.2 mm
- net +8V: track 5.19 -> 28.9 mm
- net CE-8: track 0.00 -> 21.5 mm, vias 0 -> 2
- net Ap-15: track 2.20 -> 18.0 mm
- net TEMP: track 2.76 -> 15.4 mm
- net SWDIO/TMS: track 0.00 -> 12.0 mm
- net -15V: track 0.00 -> 11.6 mm
- net -8V: track 3.90 -> 15.2 mm, vias 0 -> 2
- net SWCLK/TCLK: track 0.00 -> 11.2 mm
- net RX: track 0.00 -> 9.74 mm
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- added copper zone on B.Cu, net GND
- added copper zone on F.Cu, net GND
Other:
- board outline added: 69.9 x 48.3 mm
- board text added: "Louis DERYCKERE Romain DUHR"
- board text added: "Microcontroller & power supply unit"
